File: projects/DriverBoard/LEDDriverBoardV1.1.brd (EAGLE design)
At the start: 82.5 x 99.5 mm, 95 parts

Commit message: Updated with processor test board V2
Parts:
- moved L1_3 2.24 mm to (53.2, 70.8)
Other:
- outline, holes or cut-outs redrawn
Changed lines of the file:
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@@
 <?xml version="1.0" encoding="utf-8"?>
 <!DOCTYPE eagle SYSTEM "eagle.dtd">
-<eagle version="7.3.0">
+<eagle version="7.6.0">
 <drawing>
 <settings>
@@
 <setting verticaltext="up"/>
 </settings>
-<grid distance="0.5" unitdist="mm" unit="mm" style="lines" multiple="2" display="yes" altdistance="0.01" altunitdist="mm" altunit="mm"/>
+<grid distance="0.500000001" unitdist="mm" unit="mm" style="lines" multiple="2" display="yes" altdistance="0.00999999999" altunitdist="mm" altunit="mm"/>
 <layers>
 <layer number="1" name="Top" color="4" fill="1" visible="yes" active="yes"/>
@@
 <dimension x1="0" y1="0" x2="7" y2="99.5" x3="-23.5" y3="49.75" textsize="1.778" layer="20" dtype="vertical" unit="inch"/>
 <dimension x1="0" y1="0" x2="82.5" y2="0" x3="41.25" y3="-9.5" textsize="1.778" layer="20" dtype="vertical" unit="inch"/>
+<circle x="51.079" y="69" radius="1.2" width="0.4064" layer="20"/>
 </plain>
 <attributes>
@@
 <attribute name="VALUE" x="62.365" y="47.095" size="1.27" layer="27"/>
 </element>
-<element name="L1_3" library="Cubesat" package="SRP1245A" value="1.5u" x="54.25" y="68.75" smashed="yes" rot="R180">
-<attribute name="NAME" x="57.25" y="76.25" size="1.27" layer="21"/>
+<element name="L1_3" library="Cubesat" package="SRP1245A" value="1.5u" x="53.25" y="70.75" smashed="yes" rot="R180">
+<attribute name="NAME" x="56.25" y="78.25" size="1.27" layer="21"/>
 </element>
 <element name="D1_3" library="Cubesat" package="SMC(Z5-T)" value="" x="67" y="63" smashed="yes" rot="R270">
@@
 <wire x1="49.5" y1="78.5" x2="43.8" y2="78.5" width="1.016" layer="1"/>
 <wire x1="49.5" y1="78.5" x2="52" y2="81" width="1.016" layer="1"/>
-<wire x1="52" y1="81" x2="58.76" y2="81" width="1.016" layer="1"/>
+<wire x1="52" y1="81" x2="58.76" y2="81" width="1.2" layer="1"/>
 <wire x1="58.76" y1="81" x2="59.46" y2="81.7" width="1.016" layer="1"/>
 <contactref element="R3" pad="2"/>
