File: projects/DriverBoard/LEDDriverBoardV1.2.brd (EAGLE design)
At the start: 82.5 x 99.5 mm, 93 parts

Commit message: Updates to driverboard and driverboard library
Parts:
- added DRIVECONN2A: HARWIN_10_HORIZONTAL_SMD, LED_Driver_Board:10PINFEMALE
Connections:
- net N$10 renamed PHOTODIODE_RETURN
- net N$11 renamed IR_SDA
- net N$12 renamed IR_SCL
- net N$13 renamed IR_VDD
- net N$5 renamed LED4TEMP-
- net N$6 renamed LED1TEMP-
- net N$7 renamed LED2TEMP-
- removed net N$14: CONN13F.8, DRIVECONN2.1
- removed net N$15: CONN13F.9, DRIVECONN2.2
- removed net N$9: DRIVECONN1.5, TEMPCONN.5
- net 5V_1: no longer TEMPCONN.6
Routing:
- net N$14: track 11.0 -> 0.00 mm, vias 1 -> 0
- net N$15: track 9.92 -> 0.00 mm, vias 1 -> 0
- net N$9: track 9.33 -> 0.00 mm, vias 1 -> 0
- net 5V_1: track 26.9 -> 26.3 mm
