File: projects/DriverBoard/LEDDriverBoardV1.2.sch (EAGLE design)
At the start: 93 parts

Commit message: Updates to driverboard and driverboard library
Connections:
- net N$10 renamed PHOTODIODE_RETURN
- net N$11 renamed IR_SDA
- net N$12 renamed IR_SCL
- net N$13 renamed IR_VDD
- net N$5 renamed LED4TEMP-
- net N$6 renamed LED1TEMP-
- net N$7 renamed LED2TEMP-
- removed net N$14: CONN13F.8, DRIVECONN2.1
- removed net N$15: CONN13F.9, DRIVECONN2.2
- removed net N$9: DRIVECONN1.5, TEMPCONN.5
- net 5V_1: no longer TEMPCONN.6
Other:
- moved on the sheet: LED_MINUS_1, LED_MINUS_2, LED_MINUS_3, LED_MINUS_4, VOUT_1, VOUT_2, VOUT_3, VOUT_4
