File: projects/ControlBoard/CntrlBoardV2_0.brd (EAGLE design)
At the start: 76.2 x 76.2 mm, 106 parts

Commit message: Updated with processor test board V2
Connections:
- removed net PA12: SAMD21J.P$29
- net PA07: no longer C17.1, CH1-DM.P$5, CH2-DM.P$5, PH_AMP_2.OUT, R14.1, R34.2, TD-DM.P$7
- net PB00: now also C17.1, CH1-DM.P$5, CH2-DM.P$5, PH_AMP_2.OUT, R14.1, R34.2, TD-DM.P$7
Routing:
- net PA07: track 78.4 -> 47.0 mm, vias 6 -> 2
- net PB00: track 0.00 -> 26.5 mm, vias 0 -> 4
Changed lines of the file:
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@@
 <?xml version="1.0" encoding="utf-8"?>
 <!DOCTYPE eagle SYSTEM "eagle.dtd">
-<eagle version="7.3.0">
+<eagle version="7.6.0">
 <drawing>
 <settings>
@@
 <contactref element="SAMD21J" pad="P$2"/>
 </signal>
-<signal name="PA12">
-<contactref element="SAMD21J" pad="P$29"/>
-</signal>
 <signal name="PA24">
 <contactref element="SAMD21J" pad="P$45"/>
@@
 <signal name="PB00">
 <contactref element="SAMD21J" pad="P$61"/>
+<contactref element="R34" pad="2"/>
+<contactref element="PH_AMP_2" pad="OUT"/>
+<contactref element="CH1-DM" pad="P$5"/>
+<contactref element="TD-DM" pad="P$7"/>
+<contactref element="C17" pad="1"/>
+<contactref element="R14" pad="1"/>
+<contactref element="CH2-DM" pad="P$5"/>
+<wire x1="24.344" y1="41.35" x2="24.344" y2="43.594" width="0.3" layer="1"/>
+<wire x1="24.344" y1="43.594" x2="24.55" y2="43.8" width="0.3" layer="1"/>
+<wire x1="17.9" y1="56.965" x2="17.8" y2="60.5" width="0.3" layer="16"/>
+<wire x1="17.8" y1="60.5" x2="18.04" y2="61.15" width="0.3" layer="16"/>
+<via x="18.04" y="61.15" extent="1-16" drill="0.6"/>
+<wire x1="18.04" y1="61.15" x2="18.2" y2="60.66" width="0.3" layer="1"/>
+<wire x1="18.2" y1="60.66" x2="19.3" y2="59.6" width="0.3" layer="1"/>
+<wire x1="18.55" y1="52.5" x2="18.55" y2="53.55" width="0.3" layer="1"/>
+<wire x1="18.55" y1="53.55" x2="18.4" y2="53.7" width="0.3" layer="1"/>
+<wire x1="18.4" y1="53.7" x2="18.1" y2="54.1" width="0.3" layer="1"/>
+<wire x1="18.1" y1="54.1" x2="18.12" y2="55.12" width="0.3" layer="1"/>
+<via x="18.12" y="55.12" extent="1-16" drill="0.6"/>
+<wire x1="18.12" y1="55.12" x2="17.9" y2="55.7" width="0.3" layer="16"/>
+<wire x1="17.9" y1="55.7" x2="17.9" y2="56.965" width="0.3" layer="16"/>
+<wire x1="18.55" y1="52.5" x2="17.9" y2="51.85" width="0.3" layer="1"/>
+<wire x1="17.9" y1="51.85" x2="17.9" y2="48.8" width="0.3" layer="1"/>
+<via x="17.9" y="48.8" extent="1-16" drill="0.6"/>
+<wire x1="17.9" y1="48.8" x2="19.6" y2="47.1" width="0.3" layer="16"/>
+<wire x1="19.6" y1="47.1" x2="19.6" y2="46.6" width="0.3" layer="16"/>
+<via x="19.6" y="46.6" extent="1-16" drill="0.6"/>
+<wire x1="19.6" y1="46.6" x2="22.4" y2="43.8" width="0.3" layer="1"/>
+<wire x1="22.4" y1="43.8" x2="24.55" y2="43.8" width="0.3" layer="1"/>
+<wire x1="50.765" y1="48.55" x2="50.665" y2="55.4" width="0" layer="19" extent="1-1"/>
+<wire x1="42.34" y1="27.95" x2="50.765" y2="48.55" width="0" layer="19" extent="1-1"/>
+<wire x1="24.344" y1="41.35" x2="42.34" y2="27.95" width="0" layer="19" extent="1-1"/>
 </signal>
 <signal name="PA27">
@@
 <signal name="PA07">
 <contactref element="SAMD21J" pad="P$16"/>
-<contactref element="R34" pad="2"/>
-<contactref element="PH_AMP_2" pad="OUT"/>
-<contactref element="CH1-DM" pad="P$5"/>
-<contactref element="TD-DM" pad="P$7"/>
-<contactref element="C17" pad="1"/>
-<contactref element="R14" pad="1"/>
-<contactref element="CH2-DM" pad="P$5"/>
-<wire x1="24.344" y1="41.35" x2="24.344" y2="43.594" width="0.3" layer="1"/>
-<wire x1="24.344" y1="43.594" x2="24.55" y2="43.8" width="0.3" layer="1"/>
-<wire x1="17.9" y1="56.965" x2="17.8" y2="60.5" width="0.3" layer="16"/>
-<wire x1="17.8" y1="60.5" x2="18.04" y2="61.15" width="0.3" layer="16"/>
-<via x="18.04" y="61.15" extent="1-16" drill="0.6"/>
-<wire x1="18.04" y1="61.15" x2="18.2" y2="60.66" width="0.3" layer="1"/>
-<wire x1="18.2" y1="60.66" x2="19.3" y2="59.6" width="0.3" layer="1"/>
-<wire x1="18.55" y1="52.5" x2="18.55" y2="53.55" width="0.3" layer="1"/>
-<wire x1="18.55" y1="53.55" x2="18.4" y2="53.7" width="0.3" layer="1"/>
-<wire x1="18.4" y1="53.7" x2="18.1" y2="54.1" width="0.3" layer="1"/>
-<wire x1="18.1" y1="54.1" x2="18.12" y2="55.12" width="0.3" layer="1"/>
-<via x="18.12" y="55.12" extent="1-16" drill="0.6"/>
-<wire x1="18.12" y1="55.12" x2="17.9" y2="55.7" width="0.3" layer="16"/>
-<wire x1="17.9" y1="55.7" x2="17.9" y2="56.965" width="0.3" layer="16"/>
-<wire x1="18.55" y1="52.5" x2="17.9" y2="51.85" width="0.3" layer="1"/>
-<wire x1="17.9" y1="51.85" x2="17.9" y2="48.8" width="0.3" layer="1"/>
-<via x="17.9" y="48.8" extent="1-16" drill="0.6"/>
-<wire x1="17.9" y1="48.8" x2="19.6" y2="47.1" width="0.3" layer="16"/>
-<wire x1="19.6" y1="47.1" x2="19.6" y2="46.6" width="0.3" layer="16"/>
-<via x="19.6" y="46.6" extent="1-16" drill="0.6"/>
-<wire x1="19.6" y1="46.6" x2="22.4" y2="43.8" width="0.3" layer="1"/>
-<wire x1="22.4" y1="43.8" x2="24.55" y2="43.8" width="0.3" layer="1"/>
-<wire x1="50.665" y1="55.4" x2="49.4" y2="55.4" width="0.3" layer="1"/>
 <wire x1="49.4" y1="55.4" x2="49.16" y2="55.16" width="0.3" layer="1"/>
 <wire x1="49.16" y1="55.16" x2="49.16" y2="48.55" width="0.3" layer="1"/>
-<wire x1="49.16" y1="48.55" x2="50.765" y2="48.55" width="0.3" layer="1"/>
 <wire x1="33.09" y1="31.2" x2="33.09" y2="43.81" width="0.3" layer="1"/>
 <wire x1="33.09" y1="43.81" x2="31.6" y2="45.3" width="0.3" layer="1"/>
 <wire x1="31.6" y1="45.3" x2="26.05" y2="45.3" width="0.3" layer="1"/>
-<wire x1="26.05" y1="45.3" x2="24.55" y2="43.8" width="0.3" layer="1"/>
 <wire x1="49.16" y1="48.55" x2="48.55" y2="48.55" width="0.3" layer="1"/>
 <wire x1="48.55" y1="48.55" x2="47.5" y2="49.6" width="0.3" layer="1"/>
