File: projects/ControlBoard/CntrlBoardV3.brd (EAGLE design)
At the start: 76.2 x 76.2 mm, 144 parts, among them J1 HARWIN_06, J2 HARWIN_06, J3 M80-54006, J4 M80-54010, J5 M80-54008, J6 M80-54020, J7 M83-LMT1M2N27, J8 M80-5101005, J9 M50-3600542, M1 AON7522E, M2 SI4427BDY-T1-E3CT-ND, U1 MR25H40MDF, U10 LT6015, U11 LT6016, U12 TPS63001, U13 TPS63002, U14 MPU9250, U15 HMC5883L, U2 M24M02-DR, U3 SN74LVC1G125, U4 SN74LVC1G125, U6 MR25H40MDF, U7 AD7991-1, U8 LTC1380-GN, U9 LTC1380-GN

Commit message: Forgot to give values to 3 resistors. Doesn't impact board at all - just BOM
Parts:
- R17, R18, R19: value (none) -> 10K
Changed lines of the file:
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@@
 </element>
 <element name="R16" library="BrownSpaceEngineering" package="0805" value="10K" x="39.5" y="6.59" rot="R270"/>
-<element name="R17" library="BrownSpaceEngineering" package="0805" value="" x="50.7" y="20" rot="MR0"/>
-<element name="R18" library="BrownSpaceEngineering" package="0805" value="" x="46.81" y="20" rot="MR0"/>
-<element name="R19" library="BrownSpaceEngineering" package="0805" value="" x="43.12" y="11.7" rot="MR180"/>
+<element name="R17" library="BrownSpaceEngineering" package="0805" value="10K" x="50.7" y="20" rot="MR0"/>
+<element name="R18" library="BrownSpaceEngineering" package="0805" value="10K" x="46.81" y="20" rot="MR0"/>
+<element name="R19" library="BrownSpaceEngineering" package="0805" value="10K" x="43.12" y="11.7" rot="MR180"/>
 <element name="R2" library="BrownSpaceEngineering" package="0805" value="10K" x="39.01" y="10.87" smashed="yes" rot="R90">
 <attribute name="NAME" x="40.8791125" y="9.238340625" size="0.7112" layer="25" rot="R90"/>
