File: projects/RadioAdapterBoard/RadioAdapterBoardV4_0.brd (EAGLE design)
At the start: 31.2 x 45.5 mm, 27 parts

Commit message: Radio Adaptor Board Minor Updates
Parts:
- moved SEND 13.5 mm to (-3.25, 7.75), turned to 90 degrees
- moved CNTRLCONN 8.25 mm to (-2.86, 19.8), turned to 90 degrees
- moved LTC3112 5.13 mm to (-19.2, 28.5), flipped to the bottom, turned to 270 degrees
- moved RET 3.95 mm to (-3.25, 11.8), turned to 90 degrees
- moved C21 3.72 mm to (-20.8, 33.2)
- moved C22 3.72 mm to (-23.8, 33.2)
- moved L2 3.72 mm to (-22.2, 36.5)
- moved C14 1.60 mm to (-21.0, 6.00), flipped to the bottom
- moved C15 1.60 mm to (-21.0, 8.50), flipped to the bottom
- moved C16 1.60 mm to (-23.2, 19.8), flipped to the bottom
- moved C17 1.60 mm to (-21.0, 16.5), flipped to the bottom
- moved C18 1.60 mm to (-23.2, 16.5), flipped to the bottom
- moved C19 1.60 mm to (-28.0, 16.8), flipped to the bottom
- moved C20 1.60 mm to (-25.5, 19.8), flipped to the bottom
- moved C23 1.60 mm to (-24.2, 8.50), flipped to the bottom
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Routing:
- net P12: track 60.4 -> 0.00 mm, vias 2 -> 0
- net P2: track 40.2 -> 0.00 mm
- net P4: track 27.2 -> 0.00 mm, vias 2 -> 0
- net P29: track 25.4 -> 0.00 mm, vias 1 -> 0
- net P3: track 24.9 -> 0.00 mm
- net P14: track 24.3 -> 0.00 mm, vias 1 -> 0
- net N$1: track 131.5 -> 153.5 mm
- net 3V6-SNS: track 14.3 -> 0.00 mm, vias 1 -> 0
- net 3V6: track 13.0 -> 0.00 mm, vias 3 -> 0
- net VIN: track 8.09 -> 0.00 mm

Commit message: Radio Adaptor Board Minor Updates
Parts:
- moved SEND 28.8 mm to (-3.50, 36.5)
- moved RET 28.3 mm to (-3.50, 40.0)
- moved L2 26.8 mm to (-21.0, 9.75), turned to 90 degrees
- moved R3 25.3 mm to (-14.5, 38.0), turned to 180 degrees
- moved R12 25.3 mm to (-2.50, 9.75), turned to 270 degrees
- moved R4 25.1 mm to (-14.2, 35.2), turned to 0 degrees
- moved C21 24.2 mm to (-17.8, 9.25), turned to 180 degrees
- moved R9 23.3 mm to (-4.75, 9.50), turned to 90 degrees
- moved C22 23.0 mm to (-17.8, 11.0), turned to 180 degrees
- moved C23 21.8 mm to (-2.50, 6.50), turned to 90 degrees
- moved R8 20.2 mm to (-5.00, 12.0)
- moved R11 20.0 mm to (-6.75, 9.50)
- moved LTC3112 18.3 mm to (-10.8, 12.2)
- moved C19 17.8 mm to (-17.8, 2.25), turned to 0 degrees
- moved R6 17.2 mm to (-11.2, 6.25)
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
Commit message: Updates to the Radio Adapter Board
Parts:
- moved C19 34.8 mm to (-13.5, 36.8), flipped to the top, turned to 270 degrees
- moved PWR_ON 34.3 mm to (-2.50, 9.25), turned to 270 degrees
- moved C23 32.6 mm to (-21.8, 32.8), flipped to the top, turned to 270 degrees
- moved R5 30.2 mm to (-19.5, 32.8), flipped to the top, turned to 90 degrees
- moved R9 27.6 mm to (-24.0, 29.2), flipped to the top, turned to 270 degrees
- moved R12 27.4 mm to (-21.8, 29.2), flipped to the top, turned to 90 degrees
- moved R6 24.4 mm to (-19.5, 29.2), flipped to the top, turned to 90 degrees
- moved R8 21.7 mm to (-21.8, 25.8), flipped to the top, turned to 90 degrees
- moved R11 17.3 mm to (-24.0, 10.2), flipped to the top, turned to 0 degrees
- moved C14 17.2 mm to (-19.2, 25.0), flipped to the top, turned to 270 degrees
- moved C16 15.8 mm to (-24.0, 13.8), flipped to the top, turned to 180 degrees
- moved C18 15.5 mm to (-24.0, 12.0), flipped to the top, turned to 180 degrees
- moved R7 15.3 mm to (-22.5, 19.8), flipped to the top, turned to 90 degrees
- moved C15 15.2 mm to (-24.0, 25.8), flipped to the top, turned to 90 degrees
- moved R10 13.5 mm to (-24.8, 16.2), flipped to the top
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Connections:
- net P12: no longer PWR_ON.A
Routing:
- net FB: track 0.00 -> 30.7 mm
- net 3V6: track 0.00 -> 29.4 mm, vias 0 -> 5
- net N$26: track 0.00 -> 21.4 mm, vias 0 -> 1
- net COMP: track 0.00 -> 21.2 mm
- net N$28: track 0.00 -> 20.4 mm, vias 0 -> 1
- net N$1: track 153.5 -> 171.5 mm
- net OVP: track 0.00 -> 15.6 mm
- net N$25: track 0.00 -> 14.9 mm, vias 0 -> 1
- net N$29: track 0.00 -> 12.9 mm, vias 0 -> 1
- net VIN: track 0.00 -> 8.52 mm
- net 3V6-SNS: track 0.00 -> 7.12 mm
- net N$4: track 0.00 -> 6.51 mm
- net P3: track 0.00 -> 6.05 mm
- net N$23: track 0.00 -> 4.86 mm
- net 3V6-REF: track 0.00 -> 4.20 mm
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Other:
- board size 31.2 x 45.5 mm -> 40.2 x 45.5 mm
