File: projects/Equisat Simulator/EquisatSimulatorV1.sch (EAGLE design)
At the start: 0 parts

Commit message: BeginningofEquisatSimulator
Parts:
- added C1: 1uF, BrownSpaceEngineering:CAP0805
- added C2, C3, C4, C5, C6: 100nF, BrownSpaceEngineering:CAP0805
- added UC1: SAMD21JTQFP-64, BrownSpaceEngineering:SAMD21JTQFP-64
Connections:
- new net GND: C1.P$2, C2.P$2, C3.P$2, C4.P$2, C5.P$2, C6.P$2, UC1.GND@1, UC1.GND@2, UC1.GNDANA
- new net N$11: UC1.GND@3, UC1.GND@4
- new net VDD: C1.P$1, C2.P$1, C3.P$1, C4.P$1, C5.P$1, C6.P$1, UC1.VDDANA, UC1.VDDCORE, UC1.VDDIN, UC1.VDDIO@2, UC1.VDDIO@3
