File: projects/SolarPanels/AccessPanel/AccessPanelV3.brd (EAGLE design)
At the start: 99.5 x 99.5 mm, 49 parts

Commit message: Updates to Radio Adapter Board, Driver Board, Flash Panel. Somebody forgot to commit for a whole week or so....
Other:
- board text removed: "+Z"
Changed lines of the file:
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@@
 <board>
 <plain>
-<text x="-74.89" y="41.53" size="15" layer="20">+Y</text>
-<text x="138.24" y="48.41" size="15" layer="20">-Y</text>
-<text x="29.03" y="-37.51" size="15" layer="20">+Z</text>
-<text x="31.85" y="119.92" size="15" layer="20">-X</text>
 <wire x1="0" y1="0" x2="0" y2="8.55" width="0.4064" layer="20"/>
 <wire x1="0" y1="8.55" x2="-8.55" y2="8.55" width="0.4064" layer="20"/>
@@
 <vertex x="9.5" y="92"/>
 </polygon>
-<wire x1="22.6" y1="24.7" x2="22.6" y2="17.4" width="0.254" layer="21"/>
-<wire x1="22.6" y1="17.4" x2="42.1" y2="17.4" width="0.254" layer="21"/>
+<wire x1="26.2" y1="24.7" x2="26.2" y2="17.4" width="0.254" layer="21"/>
+<wire x1="26.2" y1="17.4" x2="42.1" y2="17.4" width="0.254" layer="21"/>
 <wire x1="42.1" y1="17.4" x2="42.1" y2="24.8" width="0.254" layer="21"/>
-<wire x1="42.1" y1="24.8" x2="22.6" y2="24.8" width="0.254" layer="21"/>
-<text x="22.9" y="17.9" size="1.016" layer="21">To
-Battery Board</text>
+<wire x1="42.1" y1="24.8" x2="26.2" y2="24.8" width="0.254" layer="21"/>
+<text x="24.7" y="18.9" size="1.016" layer="21" rot="R90">To
+Battery
+Board</text>
 <wire x1="44.8" y1="18.1" x2="60.4" y2="18.1" width="0.254" layer="21"/>
 <wire x1="60.4" y1="18.1" x2="61.2" y2="18.9" width="0.254" layer="21"/>
-<wire x1="61.2" y1="18.9" x2="61.2" y2="49.3" width="0.254" layer="21"/>
-<wire x1="61.2" y1="49.3" x2="44.8" y2="49.3" width="0.254" layer="21"/>
-<wire x1="44.8" y1="49.3" x2="44.8" y2="18.1" width="0.254" layer="21"/>
-<text x="45.5" y="46.3" size="1.016" layer="21">To
-Control Board</text>
-<text x="24.4" y="20.5" size="1.016" layer="22" rot="MR180">To
+<wire x1="61.2" y1="18.9" x2="61.2" y2="47.5" width="0.254" layer="21"/>
+<wire x1="61.2" y1="47.5" x2="44.8" y2="47.5" width="0.254" layer="21"/>
+<wire x1="44.8" y1="47.5" x2="44.8" y2="18.1" width="0.254" layer="21"/>
+<text x="44.8" y="47.8" size="1.016" layer="21">To Control Board</text>
+<text x="25.5" y="24.9" size="1.016" layer="22" rot="SMR270">To
 Battery Board</text>
-<wire x1="22.6" y1="25" x2="22.6" y2="17.4" width="0.254" layer="22"/>
-<wire x1="22.6" y1="17.4" x2="42" y2="17.4" width="0.254" layer="22"/>
+<wire x1="26.2" y1="25" x2="26.2" y2="17.4" width="0.254" layer="22"/>
+<wire x1="26.2" y1="17.4" x2="42" y2="17.4" width="0.254" layer="22"/>
 <wire x1="42" y1="17.4" x2="42" y2="25" width="0.254" layer="22"/>
-<wire x1="42" y1="25" x2="22.6" y2="25" width="0.254" layer="22"/>
+<wire x1="42" y1="25" x2="26.2" y2="25" width="0.254" layer="22"/>
 <wire x1="44.8" y1="18.1" x2="60.4" y2="18.1" width="0.254" layer="22"/>
 <wire x1="60.4" y1="18.1" x2="61.2" y2="18.9" width="0.254" layer="22"/>
-<wire x1="61.2" y1="18.9" x2="61.2" y2="49.3" width="0.254" layer="22"/>
-<wire x1="61.2" y1="49.3" x2="44.8" y2="49.3" width="0.254" layer="22"/>
-<wire x1="44.8" y1="49.3" x2="44.8" y2="18.1" width="0.254" layer="22"/>
-<text x="54.1" y="46.4" size="1.016" layer="22" rot="MR0">To
+<wire x1="61.2" y1="18.9" x2="61.2" y2="47.5" width="0.254" layer="22"/>
+<wire x1="61.2" y1="47.5" x2="44.8" y2="47.5" width="0.254" layer="22"/>
+<wire x1="44.8" y1="47.5" x2="44.8" y2="18.1" width="0.254" layer="22"/>
+<text x="60.4" y="48" size="1.016" layer="22" rot="MR0">To
 Control Board</text>
-<text x="60.8" y="53.4" size="1.016" layer="22" rot="MR0">Access Panel V3.0
+<text x="67.2" y="52.3" size="1.016" layer="22" rot="MR0">Access Panel V3.0
 BSE : EquiSat</text>
-<text x="45.4" y="51.4" size="1.016" layer="21">Access Panel V3.0
+<text x="44.5" y="51.4" size="1.016" layer="21">Access Panel V3.0
 BSE : EquiSat</text>
 <polygon width="0.254" layer="21">
-<vertex x="55.7" y="52.1"/>
+<vertex x="56.9" y="52.1"/>
 <vertex x="62.5" y="52.1"/>
 <vertex x="62.5" y="49.2"/>
-<vertex x="55.7" y="49.2"/>
+<vertex x="56.9" y="49.2"/>
 </polygon>
 <polygon width="0.254" layer="22">
 <vertex x="50.9" y="53.5"/>
-<vertex x="50.9" y="49.2"/>
-<vertex x="44.9" y="49.2"/>
-<vertex x="44.9" y="54"/>
-<vertex x="50.9" y="54"/>
+<vertex x="50.9" y="51.2"/>
+<vertex x="44.9" y="51.2"/>
+<vertex x="44.9" y="55.2"/>
+<vertex x="50.9" y="55.2"/>
 <vertex x="50.9" y="53.4"/>
 </polygon>
@@
 <text x="87.3" y="87.1" size="1.778" layer="22" rot="MR270">-Y</text>
 <text x="-5" y="87.6" size="1.778" layer="22" rot="MR270">+Y</text>
-<text x="45.5" y="54.9" size="1.016" layer="21">-Z Panel</text>
+<text x="42.6" y="56.3" size="1.016" layer="21">-Z Panel</text>
 </plain>
 <attributes>
