File: projects/ProgrammerBoard/ProgrammerBoardV1.brd (EAGLE design)
At the start: 30.1 x 31.7 mm, 14 parts, among them J9 M50-3600542

Commit message: V1
fixed a wire
Routing:
- net RESETN: track 68.9 -> 69.6 mm
Changed lines of the file:
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@@
 <contactref element="U$1" pad="B10"/>
 <contactref element="J9" pad="P6"/>
-<wire x1="3.81" y1="7.62" x2="3.81" y2="10.16" width="0.4064" layer="1"/>
-<wire x1="3.81" y1="7.62" x2="5.08" y2="6.35" width="0.4064" layer="1"/>
-<wire x1="12.7" y1="6.35" x2="5.08" y2="6.35" width="0.4064" layer="1"/>
-<wire x1="13.24" y1="8.46" x2="12.7" y2="6.35" width="0.4064" layer="1"/>
+<wire x1="12.7" y1="6.35" x2="13.24" y2="8.46" width="0.4064" layer="1"/>
 <wire x1="16.99" y1="10.16" x2="16.99" y2="17.78" width="0.4064" layer="1"/>
 <wire x1="16.99" y1="17.78" x2="19.05" y2="17.78" width="0.4064" layer="1"/>
@@
 <wire x1="17.78" y1="25.4" x2="19.05" y2="25.4" width="0.4064" layer="1"/>
 <wire x1="17.78" y1="25.4" x2="17.78" y2="23.54" width="0.4064" layer="1"/>
-<wire x1="3.81" y1="10.16" x2="6.35" y2="10.16" width="0.4064" layer="1"/>
+<wire x1="6.35" y1="10.16" x2="3.81" y2="10.16" width="0.4064" layer="1"/>
 <via x="6.35" y="10.16" extent="1-16" drill="0.6" shape="square"/>
 <wire x1="6.35" y1="27.94" x2="17.78" y2="27.94" width="0.4064" layer="16"/>
@@
 <wire x1="17.78" y1="27.94" x2="17.78" y2="25.4" width="0.4064" layer="1"/>
 <wire x1="6.35" y1="10.16" x2="6.35" y2="27.94" width="0.4064" layer="16"/>
+<wire x1="3.81" y1="10.16" x2="3.81" y2="6.35" width="0.4064" layer="1"/>
+<wire x1="3.81" y1="6.35" x2="12.7" y2="6.35" width="0.4064" layer="1"/>
 </signal>
 <signal name="UMB-CHG">
