File: projects/SolarPanels/Side Panel/SIDEPANELV5(old).brd (EAGLE design)
At the start: 99.5 x 82.5 mm, 31 parts

Commit message: side panel v5 WIP
updated cells
still figuring out cell layout
Parts:
- moved 3A 212.9 mm to (9.94, 57.9), turned to 270 degrees
- moved 3B 202.3 mm to (20.1, 56.7), turned to 90 degrees
- moved 3D 198.6 mm to (24.8, 29.4)
- moved 3C 196.5 mm to (26.8, 39.6), turned to 180 degrees
- moved IR 149.5 mm to (43.1, 13.7)
- moved C1 148.6 mm to (49.2, 13.9)
- moved PD 148.6 mm to (51.6, 15.3)
- moved 6A 127.5 mm to (79.6, 60.0)
- moved 6B 127.4 mm to (80.3, 54.0), turned to 180 degrees
- moved 6C 114.0 mm to (66.7, 43.5)
- moved 7A 111.8 mm to (93.5, 37.5), turned to 270 degrees
- moved 7C 103.6 mm to (75.5, 27.5)
- moved 7B 102.6 mm to (75.5, 35.5)
- moved 7D 101.4 mm to (50.5, 34.0), turned to 305 degrees
- moved 4B 98.6 mm to (22.0, 5.94), turned to 180 degrees
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Routing:
- net N$17: track 0.00 -> 53.9 mm
- net N$6: track 0.00 -> 44.0 mm
- net N$18: track 0.00 -> 36.2 mm
- net N$13: track 0.00 -> 32.5 mm
- net N$16: track 10.1 -> 37.0 mm
- net N$11: track 0.00 -> 25.6 mm
- net N$15: track 10.7 -> 34.5 mm
- net N$3: track 0.00 -> 23.1 mm
- net N$22: track 0.00 -> 21.8 mm
- net N$12: track 0.00 -> 20.6 mm
- net N$9: track 0.00 -> 20.5 mm
- net N$8: track 0.00 -> 19.0 mm
- net N$4: track 0.00 -> 17.9 mm
- net N$1: track 10.1 -> 26.9 mm
- net N$10: track 0.00 -> 15.1 mm
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