File: projects/BatteryTestBoard/BatteryTestBoard V1.sch (EAGLE design)
At the start: 139 parts, among them M2 IPB120P04P4L03ATMA1, SW1 BTS50015-1TAD, U1 LTC4121-4.2, U2 AD8418, U3 AD8418, U4 LC05111C13MTTTG, U5 LTC4121, U6 AP9211SA-AG-HAC-7

Commit message: Board ready for Ryan review
Parts:
- V16: value LIFE2 -> LifePo cell 2
- V17: value LIFE1 -> LifePo cell 1
- V2: value FUSE_OUT -> Fuse output
- V20: value LF_B1_OUTEN -> LifePo output enable
- V29: value LF_B1_TT -> TT
- V31: value LF_B1_OSNS -> LifePo output sense
- V32: value LF_B1_BT -> BT
- V54: value LFPOBOOST -> BOOST
- V57: value LFPOSW -> SW
- V58: value LF1_REF -> LifePo cell 1
- V59: value LF2_REF -> LifePo cell 2
- V60: value LFPOMPPT -> MPPT
- V61: value LFPOCHGSNS -> CHGSNS
- V62: value LFPOFREQ -> FREQ
- V63: value LFPOBAT -> BAT
- V65: value LFPOPROG -> PROG
- V66: value LFPOCHRG -> !CHRG
- V67: value LFPOFAULT -> !FAULT
- V68: value LFPORUN -> RUN
- V69: value LFPOINTVCC -> INTVCC
- V70: value LFPOFB -> FB
- renumbered U$3 to U7
Changed lines of the file:
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@@
 <part name="C17" library="BrownSpaceEngineering" deviceset="CAP" device="0805" value="10uF"/>
 <part name="L3" library="BrownSpaceEngineering" deviceset="IND" device="" technology="1812" value="47uH"/>
-<part name="V16" library="BrownSpaceEngineering" deviceset="VIA" device="60MIL-SQ" value="LIFE2"/>
-<part name="V17" library="BrownSpaceEngineering" deviceset="VIA" device="60MIL-SQ" value="LIFE1"/>
+<part name="V16" library="BrownSpaceEngineering" deviceset="VIA" device="60MIL-SQ" value="LifePo cell 2"/>
+<part name="V17" library="BrownSpaceEngineering" deviceset="VIA" device="60MIL-SQ" value="LifePo cell 1"/>
 <part name="C18" library="BrownSpaceEngineering" deviceset="CAP" device="0805" value="22uF"/>
-<part name="U$3" library="BrownSpaceEngineering" deviceset="VNS3NV04DP-E" device=""/>
+<part name="U7" library="BrownSpaceEngineering" deviceset="VNS3NV04DP-E" device=""/>
 <part name="R54" library="BrownSpaceEngineering" deviceset="RES" device="1210" value="34.8R@1W"/>
 <part name="R55" library="BrownSpaceEngineering" deviceset="RES" device="1210" value="34.8R@1W"/>
@@
 <part name="C25" library="BrownSpaceEngineering" deviceset="CAP" device="0805" value="150nF"/>
 <part name="GND32" library="supply1" deviceset="GND" device=""/>
-<part name="V20" library="BrownSpaceEngineering" deviceset="VIA" device="60MIL-SQ" value="LF_B1_OUTEN"/>
-<part name="V31" library="BrownSpaceEngineering" deviceset="VIA" device="60MIL-SQ" value="LF_B1_OSNS"/>
+<part name="V20" library="BrownSpaceEngineering" deviceset="VIA" device="60MIL-SQ" value="LifePo output enable"/>
+<part name="V31" library="BrownSpaceEngineering" deviceset="VIA" device="60MIL-SQ" value="LifePo output sense"/>
 <part name="V26" library="BrownSpaceEngineering" deviceset="VIA" device="-120MIL" value="LF_B1"/>
-<part name="V58" library="BrownSpaceEngineering" deviceset="VIA" device="60MIL-SQ" value="LF1_REF"/>
-<part name="V59" library="BrownSpaceEngineering" deviceset="VIA" device="60MIL-SQ" value="LF2_REF"/>
+<part name="V58" library="BrownSpaceEngineering" deviceset="VIA" device="60MIL-SQ" value="LifePo cell 1"/>
+<part name="V59" library="BrownSpaceEngineering" deviceset="VIA" device="60MIL-SQ" value="LifePo cell 2"/>
 <part name="U1" library="BrownSpaceEngineering" deviceset="LTC4121-4.2" device=""/>
 <part name="V5" library="BrownSpaceEngineering" deviceset="VIA" device="60MIL-SQ" value="GND"/>
@@
 <part name="V8" library="BrownSpaceEngineering" deviceset="VIA" device="60MIL-SQ" value="GND"/>
 <part name="V13" library="BrownSpaceEngineering" deviceset="VIA" device="60MIL-SQ" value="LF_B1_ISNS"/>
-<part name="V29" library="BrownSpaceEngineering" deviceset="VIA" device="60MIL-SQ" value="LF_B1_TT"/>
-<part name="V32" library="BrownSpaceEngineering" deviceset="VIA" device="60MIL-SQ" value="LF_B1_BT"/>
+<part name="V29" library="BrownSpaceEngineering" deviceset="VIA" device="60MIL-SQ" value="TT"/>
+<part name="V32" library="BrownSpaceEngineering" deviceset="VIA" device="60MIL-SQ" value="BT"/>
 <part name="V34" library="BrownSpaceEngineering" deviceset="VIA" device="60MIL-SQ" value="LION_IN"/>
 <part name="V35" library="BrownSpaceEngineering" deviceset="VIA" device="60MIL-SQ" value="LION_IN"/>
@@
 <part name="V53" library="BrownSpaceEngineering" deviceset="VIA" device="60MIL-SQ" value="RUN"/>
 <part name="V55" library="BrownSpaceEngineering" deviceset="VIA" device="60MIL-SQ" value="INTVCC"/>
-<part name="V54" library="BrownSpaceEngineering" deviceset="VIA" device="60MIL-SQ" value="LFPOBOOST"/>
-<part name="V57" library="BrownSpaceEngineering" deviceset="VIA" device="60MIL-SQ" value="LFPOSW"/>
-<part name="V60" library="BrownSpaceEngineering" deviceset="VIA" device="60MIL-SQ" value="LFPOMPPT"/>
-<part name="V61" library="BrownSpaceEngineering" deviceset="VIA" device="60MIL-SQ" value="LFPOCHGSNS"/>
-<part name="V62" library="BrownSpaceEngineering" deviceset="VIA" device="60MIL-SQ" value="LFPOFREQ"/>
-<part name="V63" library="BrownSpaceEngineering" deviceset="VIA" device="60MIL-SQ" value="LFPOBAT"/>
-<part name="V65" library="BrownSpaceEngineering" deviceset="VIA" device="60MIL-SQ" value="LFPOPROG"/>
-<part name="V66" library="BrownSpaceEngineering" deviceset="VIA" device="60MIL-SQ" value="LFPOCHRG"/>
-<part name="V67" library="BrownSpaceEngineering" deviceset="VIA" device="60MIL-SQ" value="LFPOFAULT"/>
-<part name="V68" library="BrownSpaceEngineering" deviceset="VIA" device="60MIL-SQ" value="LFPORUN"/>
-<part name="V69" library="BrownSpaceEngineering" deviceset="VIA" device="60MIL-SQ" value="LFPOINTVCC"/>
-<part name="V70" library="BrownSpaceEngineering" deviceset="VIA" device="60MIL-SQ" value="LFPOFB"/>
+<part name="V54" library="BrownSpaceEngineering" deviceset="VIA" device="60MIL-SQ" value="BOOST"/>
+<part name="V57" library="BrownSpaceEngineering" deviceset="VIA" device="60MIL-SQ" value="SW"/>
+<part name="V60" library="BrownSpaceEngineering" deviceset="VIA" device="60MIL-SQ" value="MPPT"/>
+<part name="V61" library="BrownSpaceEngineering" deviceset="VIA" device="60MIL-SQ" value="CHGSNS"/>
+<part name="V62" library="BrownSpaceEngineering" deviceset="VIA" device="60MIL-SQ" value="FREQ"/>
+<part name="V63" library="BrownSpaceEngineering" deviceset="VIA" device="60MIL-SQ" value="BAT"/>
+<part name="V65" library="BrownSpaceEngineering" deviceset="VIA" device="60MIL-SQ" value="PROG"/>
+<part name="V66" library="BrownSpaceEngineering" deviceset="VIA" device="60MIL-SQ" value="!CHRG"/>
+<part name="V67" library="BrownSpaceEngineering" deviceset="VIA" device="60MIL-SQ" value="!FAULT"/>
+<part name="V68" library="BrownSpaceEngineering" deviceset="VIA" device="60MIL-SQ" value="RUN"/>
+<part name="V69" library="BrownSpaceEngineering" deviceset="VIA" device="60MIL-SQ" value="INTVCC"/>
+<part name="V70" library="BrownSpaceEngineering" deviceset="VIA" device="60MIL-SQ" value="FB"/>
 <part name="U2" library="BattBoard" deviceset="AD8418" device=""/>
 <part name="U3" library="BattBoard" deviceset="AD8418" device=""/>
@@
 <part name="R22" library="BrownSpaceEngineering" deviceset="RES" device="1210" value="0R"/>
 <part name="V9" library="BrownSpaceEngineering" deviceset="VIA" device="60MIL-SQ" value="LFPO_IN"/>
-<part name="V2" library="BrownSpaceEngineering" deviceset="VIA" device="60MIL-SQ" value="FUSE_OUT"/>
+<part name="V2" library="BrownSpaceEngineering" deviceset="VIA" device="60MIL-SQ" value="Fuse output"/>
 <part name="M1" library="BrownSpaceEngineering" deviceset="AON7522E" device=""/>
 <part name="M2" library="BattBoard" deviceset="IPB120P04P4L03ATMA1" device=""/>
@@
 <instance part="V17" gate="G$1" x="66.04" y="-50.8"/>
 <instance part="C18" gate="G$1" x="25.4" y="-53.34"/>
-<instance part="U$3" gate="G$1" x="40.64" y="-73.66"/>
+<instance part="U7" gate="G$1" x="40.64" y="-73.66"/>
 <instance part="R54" gate="R$1" x="58.42" y="-55.88" smashed="yes" rot="R90">
 <attribute name="NAME" x="57.404" y="-58.42" size="1.905" layer="95" rot="R90"/>
@@
 <wire x1="106.68" y1="-104.14" x2="106.68" y2="-63.5" width="0.1524" layer="91"/>
 <junction x="106.68" y="-104.14"/>
-<pinref part="U$3" gate="G$1" pin="S2"/>
+<pinref part="U7" gate="G$1" pin="S2"/>
 <wire x1="50.8" y1="-78.74" x2="66.04" y2="-78.74" width="0.1524" layer="91"/>
 <wire x1="66.04" y1="-78.74" x2="66.04" y2="-104.14" width="0.1524" layer="91"/>
@@
 <wire x1="71.12" y1="-63.5" x2="81.28" y2="-63.5" width="0.1524" layer="91"/>
 <junction x="81.28" y="-63.5"/>
-<pinref part="U$3" gate="G$1" pin="S1"/>
+<pinref part="U7" gate="G$1" pin="S1"/>
 <wire x1="50.8" y1="-71.12" x2="73.66" y2="-71.12" width="0.1524" layer="91"/>
 <junction x="81.28" y="-71.12"/>
@@
 <net name="N$24" class="0">
 <segment>
-<pinref part="U$3" gate="G$1" pin="D1"/>
+<pinref part="U7" gate="G$1" pin="D1"/>
 <pinref part="R54" gate="R$1" pin="1"/>
 <wire x1="50.8" y1="-66.04" x2="58.42" y2="-66.04" width="0.1524" layer="91"/>
@@
 <segment>
 <pinref part="R55" gate="R$1" pin="2"/>
-<pinref part="U$3" gate="G$1" pin="D2"/>
+<pinref part="U7" gate="G$1" pin="D2"/>
 <wire x1="58.42" y1="-73.66" x2="50.8" y2="-73.66" width="0.1524" layer="91"/>
 </segment>
@@
 <net name="LF_B1_BT" class="0">
 <segment>
-<pinref part="U$3" gate="G$1" pin="G2"/>
+<pinref part="U7" gate="G$1" pin="G2"/>
 <pinref part="R57" gate="R$1" pin="2"/>
 <wire x1="33.02" y1="-76.2" x2="20.32" y2="-76.2" width="0.1524" layer="91"/>
@@
 <net name="LF_B1_TT" class="0">
 <segment>
-<pinref part="U$3" gate="G$1" pin="G1"/>
+<pinref part="U7" gate="G$1" pin="G1"/>
 <wire x1="33.02" y1="-68.58" x2="10.16" y2="-68.58" width="0.1524" layer="91"/>
 <pinref part="R56" gate="R$1" pin="2"/>
