File: projects/BatteryBoard/BatteryBoardV2B.sch (EAGLE design)
At the start: 214 parts, among them M1 BSO201SP, SW1 BTS50015-1TAD, SW2 BTS50015-1TAD, T1 AD590FLATPACK, T2 AD590FLATPACK, T3 AD590FLATPACK, T4 AD590FLATPACK, U1 TCA9535PWR, U10 LT1962-3, U11 LT1962-3, U12 LTC4411, U13 LTC4411, U14 LTC4121, U16 LTC4121, U18 AD8418, U19 AD8418, U2 AD7991-0, U3 LTC4412MPS6, U4 LTC4121-4.2, U5 LTC4121-4.2, U6 LC05111C13MTTTG, U7 LC05111C13MTTTG, U8 AD8418, U9 AD8418

Commit message: putting in correct directory
Parts:
- R12, R31: value 0.13R@1W -> 0.025R@1W
Changed lines of the file:
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@@
 <part name="LI-ION1" library="BrownSpaceEngineering" deviceset="LI-ION" device="" value="~4.1V"/>
 <part name="GND21" library="supply1" deviceset="GND" device=""/>
-<part name="R31" library="BrownSpaceEngineering" deviceset="RES" device="1210" value="0.13R@1W"/>
+<part name="R31" library="BrownSpaceEngineering" deviceset="RES" device="1210" value="0.025R@1W"/>
 <part name="R33" library="BrownSpaceEngineering" deviceset="RES" device="0805" value="150K"/>
 <part name="R34" library="BrownSpaceEngineering" deviceset="RES" device="0805" value="100K"/>
@@
 <part name="LI-ION2" library="BrownSpaceEngineering" deviceset="LI-ION" device="" value="~4.1V"/>
 <part name="GND22" library="supply1" deviceset="GND" device=""/>
-<part name="R12" library="BrownSpaceEngineering" deviceset="RES" device="1210" value="0.13R@1W"/>
+<part name="R12" library="BrownSpaceEngineering" deviceset="RES" device="1210" value="0.025R@1W"/>
 <part name="R16" library="BrownSpaceEngineering" deviceset="RES" device="0805" value="150K"/>
 <part name="R19" library="BrownSpaceEngineering" deviceset="RES" device="0805" value="100K"/>
