File: projects/BatteryBoard/BatteryBoardV2B.brd (EAGLE design)
At the start: 90.6 x 96 mm, 214 parts, among them M1 BSO201SP, SW1 BTS50015-1TAD, SW2 BTS50015-1TAD, T1 AD590FLATPACK, T2 AD590FLATPACK, T3 AD590FLATPACK, T4 AD590FLATPACK, U1 TCA9535PWR, U10 LT1962-3, U11 LT1962-3, U12 LTC4411, U13 LTC4411, U14 LTC4121, U16 LTC4121, U18 AD8418, U19 AD8418, U2 AD7991-0, U3 LTC4412MPS6, U4 LTC4121-4.2, U5 LTC4121-4.2, U6 LC05111C13MTTTG, U7 LC05111C13MTTTG, U8 AD8418, U9 AD8418

Commit message: take 4
Parts:
- moved V7 0.40 mm to (5.30, 67.5)
Changed lines of the file:
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@@
 <attribute name="NAME" x="33.76" y="53.554" size="0.7" layer="25" rot="R270"/>
 </element>
-<element name="V7" library="BrownSpaceEngineering" package="VIA-60MIL" value="5V" x="5.3" y="67.1" smashed="yes">
-<attribute name="VALUE" x="2.998" y="65.292" size="0.762" layer="27"/>
+<element name="V7" library="BrownSpaceEngineering" package="VIA-60MIL" value="5V" x="5.3" y="67.5" smashed="yes">
+<attribute name="VALUE" x="2.998" y="65.692" size="0.762" layer="27"/>
 </element>
 <element name="V8" library="BrownSpaceEngineering" package="VIA-60MIL" value="L1_TEMP" x="60.8" y="3.6" smashed="yes">
@@
 <wire x1="24.8" y1="44.9" x2="20.5" y2="49.2" width="0.2032" layer="16"/>
 <wire x1="20.5" y1="49.2" x2="8.4" y2="49.2" width="0.2032" layer="16"/>
-<wire x1="5.3" y1="63.6856625" x2="5.3" y2="67.1" width="0.2032" layer="16"/>
+<wire x1="5.3" y1="63.6856625" x2="5.3" y2="67.5" width="0.2032" layer="16"/>
 <wire x1="35.2412" y1="34.70285" x2="35.2412" y2="35.49715" width="0.2032" layer="1"/>
 <wire x1="35.2412" y1="35.49715" x2="36.94405" y2="37.2" width="0.2032" layer="1"/>
