File: projects/RomeBoard copy/RomeBoardV1.sch (EAGLE design)
At the start: 27 parts, among them J1 HEADER-5, J2 RASPBERRY-PI-HEADER, M1 2N7000, M2 2N7000, M3 2N7000

Commit message: Improved routing, added silkscreen infos
Parts:
- C2: device resistor:CPOL-EUE3.5-10 -> resistor:CPOL-EUE5-10.5
Changed lines of the file:
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@@
 <part name="GND2" library="supply1" deviceset="GND" device=""/>
 <part name="C1" library="resistor" deviceset="CPOL-EU" device="E5-10.5" value="680uF"/>
-<part name="C2" library="resistor" deviceset="CPOL-EU" device="E3.5-10" value="100uF"/>
+<part name="C2" library="resistor" deviceset="CPOL-EU" device="E5-10.5" value="100uF"/>
 <part name="LM2576" library="BrownSpaceEngineering" deviceset="LM2576" device="HEATSINK" value="LM2576HEATSINK"/>
 <part name="D1" library="BrownSpaceEngineering" deviceset="1N5820" device=""/>
