File: projects/RomeBoard/RomeBoardV1.1B.brd (EAGLE design)
At the start: 120 x 150 mm, 36 parts, among them J1 HEADER-5, J2 RASPBERRY-PI-HEADER, M1 ZVN4424A, M2 ZVN4424A, M3 ZVN4424A, U1 LM1084IT-ADJ

Commit message: final version of 1.1B (pending very minor changes)
Parts:
- added V3: GND, BrownSpaceEngineering:VIA-60MIL
- R3: value 100R -> 200R
- R4: value 75R -> 150R
- R5, R6, R7: value 147R -> 300R
- V1, V2: device BrownSpaceEngineering:VIA-120MIL -> BrownSpaceEngineering:VIA-60MIL
- moved FAN2 9.50 mm to (91.5, 97.0)
- moved R8 9.00 mm to (91.5, 79.0)
- moved C5 8.00 mm to (91.5, 93.5)
- moved C4 6.50 mm to (91.5, 122.5)
- moved FAN1 5.00 mm to (91.5, 126.0)
- moved J1 5.00 mm to (103.0, 143.5)
- moved V2 5.00 mm to (5.00, 63.5)
- moved V1 3.00 mm to (5.00, 69.0)
Connections:
- net 3V3: now also J2.P17
- net GND: now also V3.P$1
Routing:
- net 3V3: track 15.2 -> 36.6 mm
- net !SHDN: track 100.0 -> 93.0 mm
- net TX_D: track 108.8 -> 103.4 mm, vias 1 -> 3
- net RX_D: track 113.9 -> 108.9 mm
- net GND: vias 142 -> 193
Other:
- board size 120 x 150 mm -> 120 x 155 mm
- board text added: "HDMI Out"
- board text added: "USB Power In"
- board text added: "board design by M. Kohli"
- board text removed: "M. Kohli - Brown U. class of 2018"

Commit message: Silkscreen + Via
Parts:
- added V6: !SHDN, BrownSpaceEngineering:VIA-60MIL
- moved V2 2.50 mm to (3.50, 65.5)
- moved V3 2.12 mm to (3.50, 56.5)
- moved V1 1.58 mm to (3.50, 69.5)
Connections:
- net !SHDN: now also V6.P$1
Routing:
- net !SHDN: track 93.0 -> 166.5 mm
- net TX_D: track 103.4 -> 104.7 mm
- net RX_D: track 108.9 -> 109.6 mm
Other:
- board text added: "Viviana Arrunategui Mckenna Cisler Tyler Fox Manav Kohli Teijiro Nishimura Caelan Ritter"
- board text added: "board design by M. Kohli '18"
- board text removed: "Viviana Arrunategui Mckenna Cisler Tyler Fox Manav Kohli Caelan Ritter"
- board text removed: "board design by M. Kohli"
