File: projects/RomeBoard/RomeBoardV1.2.brd (EAGLE design)
At the start: 120 x 164.5 mm, 38 parts, among them J2 RASPBERRY-PI-HEADER, M1 ZVN4424A, M2 ZVN4424A, M3 ZVN4424A, U1 LM1084IT-ADJ

Commit message: Rome Board v1.2 updates
Parts:
- X1: device con-yamaichi:USB-A003 -> con-berg:PN87520
- moved X1 10.0 mm to (103.5, 146.5)
Changed lines of the file:
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@@
 <hole x="115" y="159.5" drill="2.844"/>
 <text x="23.5" y="158.5" size="3.2" layer="51" font="vector" ratio="19">BROWN SPACE ENGINEERING GROUND STATION</text>
-<text x="99.5" y="145.5" size="1.27" layer="51" font="vector" ratio="13">Pi Power</text>
+<text x="100" y="139.5" size="1.27" layer="51" font="vector" ratio="13">Pi Power</text>
 <text x="107" y="116" size="2.2" layer="51" font="vector" ratio="16" align="center">Brown U.
 Providence, R.I.
@@
 <attribute name="VALUE" x="5" y="59" size="1.016" layer="27" font="vector" ratio="13"/>
 </element>
-<element name="X1" library="con-yamaichi" library_urn="urn:adsk.eagle:library:202" package="USB-A003" package3d_urn="urn:adsk.eagle:package:11805/1" value="" x="103.5" y="156.5" rot="R180">
-<attribute name="MF" value="" x="103.5" y="156.5" size="1.778" layer="27" rot="R180" display="off"/>
-<attribute name="MPN" value="" x="103.5" y="156.5" size="1.778" layer="27" rot="R180" display="off"/>
-<attribute name="OC_FARNELL" value="unknown" x="103.5" y="156.5" size="1.778" layer="27" rot="R180" display="off"/>
-<attribute name="OC_NEWARK" value="unknown" x="103.5" y="156.5" size="1.778" layer="27" rot="R180" display="off"/>
+<element name="X1" library="con-berg" library_urn="urn:adsk.eagle:library:130" package="PN87520" package3d_urn="urn:adsk.eagle:package:6146/1" value="" x="103.5" y="146.5" rot="R180">
+<attribute name="MF" value="" x="103.5" y="146.5" size="1.778" layer="27" rot="R180" display="off"/>
+<attribute name="MPN" value="" x="103.5" y="146.5" size="1.778" layer="27" rot="R180" display="off"/>
+<attribute name="OC_FARNELL" value="unknown" x="103.5" y="146.5" size="1.778" layer="27" rot="R180" display="off"/>
+<attribute name="OC_NEWARK" value="unknown" x="103.5" y="146.5" size="1.778" layer="27" rot="R180" display="off"/>
 </element>
 </elements>
@@
 <wire x1="14.25" y1="4.94" x2="10.5" y2="11" width="0" layer="19" extent="1-1"/>
 <wire x1="44.96" y1="15.5" x2="36" y2="19" width="0" layer="19" extent="1-1"/>
+<wire x1="100" y1="143.79" x2="14.25" y2="4.94" width="0" layer="19" extent="1-1"/>
+<wire x1="102.5" y1="143.79" x2="100" y2="143.79" width="0" layer="19" extent="1-1"/>
+<wire x1="104.5" y1="143.79" x2="102.5" y2="143.79" width="0" layer="19" extent="1-1"/>
 <wire x1="53.5" y1="9" x2="44.96" y2="15.5" width="0" layer="19" extent="1-1"/>
 <wire x1="55" y1="9" x2="53.5" y2="9" width="0" layer="19" extent="1-1"/>
 <wire x1="56.5" y1="9" x2="55" y2="9" width="0" layer="19" extent="1-1"/>
-<wire x1="100" y1="142.5" x2="3" y2="11" width="0" layer="19" extent="1-1"/>
-<wire x1="102.5" y1="142.5" x2="100" y2="142.5" width="0" layer="19" extent="1-1"/>
-<wire x1="104.5" y1="142.5" x2="102.5" y2="142.5" width="0" layer="19" extent="1-1"/>
 <wire x1="88.5" y1="20.27" x2="56.5" y2="9" width="0" layer="19" extent="1-1"/>
 <wire x1="90.5" y1="13.08" x2="88.5" y2="20.27" width="0" layer="19" extent="1-1"/>
@@
 <wire x1="113" y1="17" x2="113" y2="18.5" width="0" layer="19" extent="1-1"/>
 <wire x1="111.5" y1="17" x2="110" y2="17" width="0" layer="19" extent="1-1"/>
+<polygon width="0.1524" layer="1">
+<vertex x="98.5" y="145.5"/>
+<vertex x="98.5" y="142"/>
+<vertex x="105.5" y="142"/>
+<vertex x="105.5" y="145.5"/>
+</polygon>
 </signal>
 <signal name="3V6">
@@
 <wire x1="88.5" y1="17.73" x2="91.8" y2="22" width="0" layer="19" extent="16-16"/>
 <wire x1="80" y1="14.04" x2="88.5" y2="17.73" width="0" layer="19" extent="1-1"/>
+<wire x1="107" y1="143.79" x2="5" y2="16.92" width="0" layer="19" extent="1-1"/>
 <wire x1="54" y1="5" x2="80" y2="14.04" width="0" layer="19" extent="1-1"/>
-<wire x1="107" y1="142.5" x2="2.5" y2="19.42" width="0" layer="19" extent="1-16"/>
 </signal>
 <signal name="TX_L">

Commit message: Rome board v1.2 updates
Routing:
- net !SHDN: track 164.7 -> 165.6 mm
Changed lines of the file:
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@@
 <wire x1="54.5" y1="41" x2="59" y2="41" width="0.254" layer="1"/>
 <wire x1="54" y1="43.13" x2="54" y2="41.5" width="0.254" layer="1"/>
-<wire x1="72.3054" y1="54.3054" x2="59" y2="41" width="0.254" layer="1"/>
+<wire x1="59" y1="41" x2="72.3054" y2="54.3054" width="0.254" layer="1"/>
 <wire x1="61.35" y1="77.77" x2="60.85" y2="77.77" width="0.254" layer="1"/>
-<wire x1="72.3054" y1="54.3054" x2="72.3054" y2="78.28553125" width="0.254" layer="1"/>
-<wire x1="60.85" y1="77.77" x2="60.85" y2="80.85" width="0.254" layer="1"/>
-<wire x1="60.85" y1="80.85" x2="62" y2="83.5" width="0.254" layer="1"/>
 <wire x1="90.92" y1="83.5" x2="91.5" y2="84.08" width="0.254" layer="1"/>
-<wire x1="62" y1="83.5" x2="72.01986875" y2="83.5" width="0.254" layer="1"/>
-<wire x1="72.01986875" y1="83.5" x2="90.92" y2="83.5" width="0.254" layer="1"/>
-<wire x1="72.3054" y1="78.28553125" x2="72.01986875" y2="83.5" width="0.254" layer="1"/>
+<wire x1="72.5" y1="83.5" x2="90.92" y2="83.5" width="0.254" layer="1"/>
 <contactref element="V6" pad="P$1"/>
 <wire x1="3.5" y1="61" x2="1.5" y2="63" width="0.254" layer="1"/>
@@
 <wire x1="55.30526875" y1="76.5254" x2="58.82553125" y2="76.5254" width="0.254" layer="1"/>
 <wire x1="27.5" y1="73" x2="52.76013125" y2="73" width="0.254" layer="1"/>
+<wire x1="72.3054" y1="83.3054" x2="72.5" y2="83.5" width="0.1524" layer="1"/>
+<wire x1="60.85" y1="83.35" x2="61" y2="83.5" width="0.254" layer="1"/>
+<wire x1="60.85" y1="77.77" x2="60.85" y2="83.35" width="0.254" layer="1"/>
+<wire x1="61" y1="83.5" x2="72.5" y2="83.5" width="0.254" layer="1"/>
+<wire x1="72.3054" y1="54.3054" x2="72.3054" y2="83.3054" width="0.254" layer="1"/>
 </signal>
 <signal name="TX_D">
@@
 <wire x1="113" y1="17" x2="113" y2="18.5" width="0" layer="19" extent="1-1"/>
 <wire x1="111.5" y1="17" x2="110" y2="17" width="0" layer="19" extent="1-1"/>
-<polygon width="0.1524" layer="1">
-<vertex x="98.5" y="145.5"/>
-<vertex x="98.5" y="142"/>
+<polygon width="0.1524" layer="1" thermals="no">
+<vertex x="99" y="145.5"/>
+<vertex x="99" y="142"/>
 <vertex x="105.5" y="142"/>
 <vertex x="105.5" y="145.5"/>

Commit message: Silkscreen tweaks
Other:
- board text added: ""Sloth on the Moon", a.k.a. Sid Pedro Dionísio"
- board text added: "Brown U. Providence, R.I. U.S.A. V1.2 July 2018"
- board text added: "Viviana Arrunategui Mckenna Cisler Tyler Fox Manav Kohli Teijiro Nishimura Caelan Ritter Andrew Duncombe"
- board text removed: "Brown U. Providence, R.I. U.S.A. V1.1 April 2018"
- board text removed: "Viviana Arrunategui Mckenna Cisler Tyler Fox Manav Kohli Teijiro Nishimura Caelan Ritter"
- board text removed: "board design by M. Kohli '18"
